File: Cable Detector module.kicad_sch (KiCad schematic)
At the start: 12 parts, among them J1 INPUT, Q1 BC547, U1 CA3130

Commit message: Cable Detector Module is renewed
Other:
- company: (none) -> by Muxtar_Safarov
- title: (none) -> Cable Detector Module 
Changed lines of the file:
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@@
 (kicad_sch (version 20230121) (generator eeschema)
   (paper "A4")
+  (title_block
+    (title "Cable Detector Module ")
+    (date "12.10.2022")
+    (rev "1.0")
+    (company "by Muxtar_Safarov")
+  )
   (junction (at 139.7 86.36) (diameter 0) (color 0 0 0 0)
   )
